File: WH-MDC05F3E5_comm/eagle/WH-MDC05F3E5_comm_v3.0.sch (EAGLE design)
At the start: 30 parts, among them IC1 4011D, IC2 4066D, IC3 4011D, T1 BC846ASMD, T2 BC846ASMD

Commit message: change to previous version: - added pin 1 chamfer notice in schematics - added link to a suitable USB2serial converter - additional pictures
Other:
- note added: "Pin 1 Markierung: Das IC 4011D hat keine Pin 1 Markierung, sondern auf der langen Seite des Gehäuses eine abgeschrägte Kante. Diese markiert (links) den Pin 1."
Changed lines of the file:
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@@
 oder kompatibel (mit RTS, 960 bd)</text>
 <wire x1="264.16" y1="180.34" x2="264.16" y2="35.56" width="0.1524" layer="95"/>
-<wire x1="0" y1="35.56" x2="203.2" y2="35.56" width="0.1524" layer="95"/>
 <wire x1="205.74" y1="35.56" x2="264.16" y2="35.56" width="0.1524" layer="95"/>
 <wire x1="203.2" y1="68.58" x2="203.2" y2="55.88" width="0.1524" layer="95"/>
@@
 ein eigenes Paket gesendet</text>
 <text x="12.7" y="38.1" size="1.778" layer="95">nicht verwendete Gatter</text>
+<text x="12.7" y="22.86" size="1.778" layer="95">Pin 1 Markierung:
+Das IC 4011D hat keine Pin 1 Markierung,
+sondern auf der langen Seite des Gehäuses
+eine abgeschrägte Kante. Diese markiert
+(links) den Pin 1.</text>
 </plain>
 <instances>
